Commit message: fix simulation  issues; robot seems to raise leg fine

File: src/unitree_ros/go1_description/xacro/gazebo.xacro (robot description, xacro)
@@ -20,5 +20,5 @@
     </gazebo>
     <!-- Show the trajectory of foot. You can add another trajectory about another foot. -->
-    <!-- <gazebo>
+    <gazebo>
         <plugin name="3dplot" filename="libLinkPlot3DPlugin.so">
             <frequency>100</frequency>
@@ -29,5 +29,5 @@
             </plot>
         </plugin>
-    </gazebo> -->
+    </gazebo>
     <gazebo>
         <plugin filename="libgazebo_ros_force.so" name="gazebo_ros_force">
@@ -55,116 +55,4 @@
         </sensor>
     </gazebo>
-    <!-- Depth camera -->
-    <!-- <gazebo>
-        <plugin name="camera_plugin" filename="libgazebo_ros_openni_kinect.so">
-            <baseline>0.025</baseline>
-            <always_on>true</always_on>
-            <updateRate>0.0</updateRate>
-            <cameraName>unitree_camera_left</cameraName>
-            <frameName>depthCamera_link_left</frameName>
-            <imageTopicName>rgb/imageRaw_left</imageTopicName>
-            <depthImageTopicName>depth/imageRaw_left</depthImageTopicName>
-            <pointCloudTopicName>depth/points_left</pointCloudTopicName>
-            <cameraInfoTopicName>rgb/cameraInfo_left</cameraInfoTopicName>
-            <depthImageCameraInfoTopicName>depth/cameraInfo_left</depthImageCameraInfoTopicName>
-            <pointCloudCutoff>0.1</pointCloudCutoff>
-            <pointCloudCutoffMax>1.5</pointCloudCutoffMax>
-            <distortionK1>0.0</distortionK1>
-            <distortionK2>0.0</distortionK2>
-            <distortionK3>0.0</distortionK3>
-            <distortionT1>0.0</distortionT1>
-            <distortionT2>0.0</distortionT2>
-            <CxPrime>0.0</CxPrime>
-            <Cx>0.0045</Cx>
-            <Cy>0.0039</Cy>
-            <focalLength>0.004</focalLength>
-            <hackBaseline>0.0</hackBaseline>
-        </plugin>
-    </gazebo> -->
-    <!-- <gazebo reference="depthCamera_link_left">
-        <sensor name="unitree_camera_left" type="depth_camera">
-            <update_rate>16</update_rate>
-            <always_on>true</always_on>
-            <visualize>true</visualize>
-            <camera>
-                <horizontal_fov>2.094</horizontal_fov>
-                <image>
-                    <width>928</width>
-                    <height>800</height>
-                    <format>R8G8B8</format>
-                </image>
-                <depth_camera></depth_camera>
-                <clip>
-                    <near>0.1</near>
-                    <far>100</far>
-                </clip>
-            </camera>
-            <plugin name="camera_plugin" filename="libgazebo_ros_openni_kinect.so">
-                <baseline>0.025</baseline>
-                <always_on>true</always_on>
-                <updateRate>0.0</updateRate>
-                <cameraName>unitree_camera_left</cameraName>
-                <frameName>depthCamera_link_left</frameName>
-                <imageTopicName>rgb/imageRaw_left</imageTopicName>
-                <depthImageTopicName>depth/imageRaw_left</depthImageTopicName>
-                <pointCloudTopicName>depth/points_left</pointCloudTopicName>
-                <cameraInfoTopicName>rgb/cameraInfo_left</cameraInfoTopicName>
-                <depthImageCameraInfoTopicName>depth/cameraInfo_left</depthImageCameraInfoTopicName>
-                <pointCloudCutoff>0.1</pointCloudCutoff>
-                <pointCloudCutoffMax>1.5</pointCloudCutoffMax>
-                <distortionK1>0.0</distortionK1>
-                <distortionK2>0.0</distortionK2>
-                <distortionK3>0.0</distortionK3>
-                <distortionT1>0.0</distortionT1>
-                <distortionT2>0.0</distortionT2>
-                <CxPrime>0.0</CxPrime>
-                <Cx>0.0045</Cx>
-                <Cy>0.0039</Cy>
-                <focalLength>0.004</focalLength>
-                <hackBaseline>0.0</hackBaseline>
-            </plugin>
-        </sensor>
-    </gazebo> -->
-  <gazebo reference="depthCamera_link_left">
-    <sensor name="camera_link_camera" type="depth">
-      <update_rate>20</update_rate>
-      <camera>
-        <horizontal_fov>1.047198</horizontal_fov>
-        <image>
-          <width>640</width>
-          <height>480</height>
-          <format>R8G8B8</format>
-        </image>
-        <clip>
-          <near>0.05</near>
-          <far>3</far>
-        </clip>
-      </camera>
-      <plugin name="camera_link_controller" filename="libgazebo_ros_openni_kinect.so">
-        <baseline>0.2</baseline>
-        <alwaysOn>true</alwaysOn>
-        <updateRate>1.0</updateRate>
-        <cameraName>camera_link_ir</cameraName>
-        <imageTopicName>/camera_link/color/image_raw</imageTopicName>
-        <cameraInfoTopicName>/camera_link/color/camera_info</cameraInfoTopicName>
-        <depthImageTopicName>/camera_link/depth/image_raw</depthImageTopicName>
-        <depthImageInfoTopicName>/camera_link/depth/camera_info</depthImageInfoTopicName>
-        <pointCloudTopicName>/camera_link/depth/points</pointCloudTopicName>
-        <frameName>depthCamera_link_left</frameName>
-        <pointCloudCutoff>0.5</pointCloudCutoff>
-        <pointCloudCutoffMax>3.0</pointCloudCutoffMax>
-        <distortionK1>0.00000001</distortionK1>
-        <distortionK2>0.00000001</distortionK2>
-        <distortionK3>0.00000001</distortionK3>
-        <distortionT1>0.00000001</distortionT1>
-        <distortionT2>0.00000001</distortionT2>
-        <CxPrime>0</CxPrime>
-        <Cx>0</Cx>
-        <Cy>0</Cy>
-        <focalLength>0</focalLength>
-        <hackBaseline>0</hackBaseline>
-      </plugin>
-    </sensor>
-  </gazebo>
     <!-- Foot contacts. -->
     <gazebo reference="FR_calf">

File: src/unitree_ros/go1_description/xacro/robot.xacro (robot description, xacro)
@@ -5,10 +5,5 @@
     <xacro:include filename="$(find go1_description)/xacro/materials.xacro"/>
     <xacro:include filename="$(find go1_description)/xacro/leg.xacro"/>
-    <!-- <xacro:include filename="$(find go1_description)/xacro/stairs.xacro"/> -->
     <xacro:include filename="$(find go1_description)/xacro/gazebo.xacro"/>
-    <xacro:include filename="$(find go1_description)/xacro/depthCamera.xacro"/>
-    <xacro:include filename="$(find go1_description)/xacro/ultraSound.xacro"/>
-    <!-- <xacro:include filename="$(find go1_gazebo)/launch/stairs.urdf.xacro"/> -->
-    <!-- <xacro:stairs stairs="15" xpos="0" ypos="0" zpos="0" /> -->
     <!-- Rotor related joint and link is only for demonstrate location. -->
     <!-- Actually, the rotor will rotate and the joint is not fixed. Reduction ratio should be considered. -->
@@ -87,41 +82,3 @@
     <xacro:leg name="RR" mirror="-1" mirror_dae="False"  front_hind="-1" front_hind_dae="False" />
     <xacro:leg name="RL" mirror="1"  mirror_dae="True"   front_hind="-1" front_hind_dae="False" />
-    <xacro:depthCamera camID="1" name="face">
-        <origin rpy="${PI} 0 0" xyz="0.2785 0.0125 0.0167"/>
-    </xacro:depthCamera>
-    <xacro:depthCamera camID="2" name="chin">
-        <origin rpy="${PI} ${PI/2} 0" xyz="0.2522 0.0125 -0.0436"/>
-    </xacro:depthCamera>
-    <xacro:depthCamera camID="3" name="left">
-        <origin rpy="${PI} 0.2618 ${PI/2}" xyz="-0.066 0.082 -0.0176"/>
-    </xacro:depthCamera>
-    <xacro:depthCamera camID="4" name="right">
-        <origin rpy="${PI} 0.2618 ${-PI/2}" xyz="-0.041 -0.082 -0.0176"/>
-    </xacro:depthCamera>
-    <xacro:depthCamera camID="5" name="rearDown">
-        <origin rpy="${PI} ${PI/2} 0" xyz="-0.0825 0.0125 -0.04365"/>
-    </xacro:depthCamera>
-    <joint name="camera_laserscan_joint_left" type="fixed">
-        <origin rpy="0 0.2618 0" xyz="0 0 0"/>
-        <parent link="camera_left"/>
-        <child link="camera_laserscan_link_left"/>
-    </joint>
-    <link name="camera_laserscan_link_left">
-    </link>
-    <joint name="camera_laserscan_joint_right" type="fixed">
-        <origin rpy="0 0.2618 0" xyz="0 0 0"/>
-        <parent link="camera_right"/>
-        <child link="camera_laserscan_link_right"/>
-    </joint>
-    <link name="camera_laserscan_link_right">
-    </link>
-    <xacro:ultraSound name="left">
-        <origin rpy="0 0.2618 ${PI/2}" xyz="-0.0535  0.0826 0.00868"/>
-    </xacro:ultraSound>
-    <xacro:ultraSound name="right">
-        <origin rpy="0 0.2618 ${-PI/2}" xyz="-0.0535 -0.0826 0.00868"/>
-    </xacro:ultraSound>
-    <xacro:ultraSound name="face">
-        <origin rpy="0 0 0" xyz="0.2747 0.0 -0.0088"/>
-    </xacro:ultraSound>
 </robot>
